File: Kicad files/buck-converter-8A.kicad_sch (KiCad schematic)
At the start: 1 part, among them U1 TPS54821RHLR

Commit message: full schematics done
Parts:
- added C1, C2, C50: 100nf, symbol Device:C
- added C10, C11, C12, C13, C14, C15, C19, C20, C21, C22, C23, C24, C25, C51, C6, C7, C8, C9: 10uf, symbol Device:C
- added C3: 10pf, symbol Device:C
- added C4: 20p, symbol Device:C
- added C5: 2n2f, symbol Device:C
- added J1, J3: Screw_01x02, symbol Connector:Screw_Terminal_01x02
- added L3: IHLP5050EZER4R7M01, Inductor_SMD:L_Sunlord_SWPA5040S, symbol Device:L
- added R1: 47k, symbol Device:R
- added R2: 90k9, symbol Device:R
- added R3: 10k, symbol Device:R
- added R31: 5k1, symbol Device:R
- added R32: 33K2, symbol Device:R
- added R4: 22k, symbol Device:R
Connections:
- net PVIN is gone; now on net +VIN: U1.4 (PVIN), U1.5 (PVIN)
- net GND: now also C1.1, C10.1, C11.1, C12.1, C13.1, C14.1, C15.1, C19.1, C20.1, C21.1, C22.1, C23.1, C24.1, C25.1, C4.1, C5.1, C6.1, C7.1, C8.1, C9.1, J1.1 (Pin_1), J3.1 (Pin_1), R1.2, R3.2
- net RT/CLK: now reaches U1.1 (RT/CLK)
- net RT/CLK: now also R1.1
- net PH: now reaches U1.11 (PH), U1.12 (PH)
- net PH: now also C2.2, L3.1
- net BOOT: now reaches U1.13 (BOOT)
- net BOOT: now also C2.1
- net +VIN: now reaches U1.6 (VIN)
- net +VIN: now also C10.2, C11.2, C12.2, C13.2, C14.2, C15.2, C6.2, C7.2, C8.2, C9.2, J3.2 (Pin_2)
- net VSENSE: now reaches U1.7 (VSENSE)
- net VSENSE: now also C3.1, R2.2, R3.1
- net COMP: now reaches U1.8 (COMP)
- net COMP: now also C4.2, R4.1
- net SS/TR: now reaches U1.9 (SS/TR)
- net SS/TR: now also C1.2
- new net +6V: C19.2, C20.2, C21.2, C22.2, C23.2, C24.2, C25.2, C3.2, J1.2 (Pin_2), L3.2, R2.1
- new net COMP_MID: C5.2, R4.2
- no-connect marks 0 -> 1
Other:
- note added: "CAPACITORS"
- note added: "INPUT CAPACITORS"
- note added: "INPUT CONNECTOR"
- note added: "OUTPUT CAPACITORS"
- note added: "OUTPUT CONNECTOR"
- note added: "POWER CONNECTORS"
- note added: "TPS54821RHLR"
- moved on the sheet: U1

Commit message: full schematics done
Parts:
- removed C50: 100nf, symbol Device:C
- removed C51: 10uf, symbol Device:C
- removed R31: 5k1, symbol Device:R
- removed R32: 33K2, symbol Device:R
