File: Kicad files/buck-converter-8A.kicad_sch (KiCad schematic)
At the start: 30 parts, among them J20 Screw_01x02, J21 Screw_01x02, U12 TPS54821RHLR

Commit message: pcb is done
Parts:
- C1: renamed from C102; footprint (none) -> Capacitor_SMD:C_0603_1608Metric
- C10: renamed from C111; footprint (none) -> Capacitor_SMD:C_0603_1608Metric
- C11: renamed from C112; footprint (none) -> Capacitor_SMD:C_0603_1608Metric
- C12: renamed from C113; footprint (none) -> Capacitor_SMD:C_0603_1608Metric
- C13: renamed from C114; footprint (none) -> Capacitor_SMD:C_0603_1608Metric
- C14: renamed from C115; footprint (none) -> Capacitor_SMD:C_0603_1608Metric
- C15: renamed from C116; footprint (none) -> Capacitor_SMD:C_0603_1608Metric
- C16: renamed from C117; footprint (none) -> Capacitor_SMD:C_0603_1608Metric
- C17: renamed from C118; footprint (none) -> Capacitor_SMD:C_0603_1608Metric
- C18: renamed from C119; footprint (none) -> Capacitor_SMD:C_0603_1608Metric
- C19: renamed from C120; footprint (none) -> Capacitor_SMD:C_0603_1608Metric
- C2: renamed from C103; footprint (none) -> Capacitor_SMD:C_0603_1608Metric
- C20: renamed from C121; footprint (none) -> Capacitor_SMD:C_0603_1608Metric
- C21: renamed from C122; footprint (none) -> Capacitor_SMD:C_0603_1608Metric
- C22: renamed from C123; footprint (none) -> Capacitor_SMD:C_0603_1608Metric
- C3: renamed from C104; footprint (none) -> Capacitor_SMD:C_0603_1608Metric
- C4: renamed from C105; footprint (none) -> Capacitor_SMD:C_0603_1608Metric
- C5: renamed from C106; footprint (none) -> Capacitor_SMD:C_0603_1608Metric
- C6: renamed from C107; footprint (none) -> Capacitor_SMD:C_0603_1608Metric
- C7: renamed from C108; footprint (none) -> Capacitor_SMD:C_0603_1608Metric
- C8: renamed from C109; footprint (none) -> Capacitor_SMD:C_0603_1608Metric
- C9: renamed from C110; footprint (none) -> Capacitor_SMD:C_0603_1608Metric
- J1: renamed from J20; footprint (none) -> TerminalBlock_RND:TerminalBlock_RND_205-00045_1x02_P5.00mm_Horizontal
- J2: renamed from J21; footprint (none) -> TerminalBlock_RND:TerminalBlock_RND_205-00045_1x02_P5.00mm_Horizontal
- L1: renamed from L6; value IHLP5050EZER4R7M01 -> IHLP5050EZER4R7M01 4u7h; footprint Inductor_SMD:L_Sunlord_SWPA5040S -> IHLP5050EZER4R7M01:IHLP5050EZER4R7M01
- R1: renamed from R82; footprint (none) -> Resistor_SMD:R_0603_1608Metric
- R2: renamed from R83; footprint (none) -> Resistor_SMD:R_0603_1608Metric
- R3: renamed from R84; footprint (none) -> Resistor_SMD:R_0603_1608Metric
- R4: renamed from R85; footprint (none) -> Resistor_SMD:R_0603_1608Metric
- renumbered U12 to U1
Connections:
- net +6V: now also J2.1 (Pin_1); no longer J2.2 (Pin_2)
- net GND: now also J2.2 (Pin_2); no longer J2.1 (Pin_1)
Other:
- moved on the sheet: C1, C2, C4, J2, L1, R1, R3, R4, U1
