File: Kicad files/buck-converter-8A.kicad_pcb (KiCad board)
At the start: 2 copper layers, 62 x 18 mm, 31 parts, among them J1 Screw_01x02, J2 Screw_01x02, U1 TPS54821RHLR

Commit message: final changes
Parts:
- added G***: LOGO, LOGO, F.Cu at (125.2, 96.3)
- added G***: LOGO, LOGO, B.Cu at (136.5, 85.0)
- added G***: LOGO, LOGO, B.Cu at (160.2, 93.8)
Other:
- board text added: "{dblquote}FOLLOW THE WHITE RABBIT...{dblquote}"
- board text added: "{dblquote}ONE SHALL STAND, ONE SHALL FALL{dblquote}"
